Commit message: Update

File: body.urdf (robot description, URDF)
Before this commit: robot robot, 10 links, 9 joints
Links:
- removed link BackLeft
- removed link BackLowerLeft
- removed link BackLowerRight
- removed link BackRight
- removed link FrontLeft
- removed link FrontLowerLeft
- removed link FrontLowerRight
- removed link FrontRight
- removed link Torso
- added link 0, mass 1; collision box size=2.699314353951913 1.8787204679229959 0.7886445005323207; visual box size=2.699314353951913 1.8787204679229959 0.7886445005323207
- added link 1, mass 1; collision box size=1.8775634867757782 0.4942450834240525 0.7222432616709291; visual box size=1.8775634867757782 0.4942450834240525 0.7222432616709291
- added link 2, mass 1; collision box size=2.0000962611517035 1.8934834306146064 1.8432109526216272; visual box size=2.0000962611517035 1.8934834306146064 1.8432109526216272
- added link 3, mass 1; collision box size=0.9833127699007228 2.858447423223876 2.32288305471027; visual box size=0.9833127699007228 2.858447423223876 2.32288305471027
- link Head: geometry collision box size=0.3409802625745797 0.329978758192523 2.4535335801865568; visual box size=0.3409802625745797 0.329978758192523 2.4535335801865568
Joints:
- removed joint BackLeft_BackLowerLeft
- removed joint BackRight_BackLowerRight
- removed joint FrontLeft_FrontLowerLeft
- removed joint FrontRight_FrontLowerRight
- removed joint Torso_BackLeft
- removed joint Torso_BackRight
- removed joint Torso_FrontLeft
- removed joint Torso_FrontRight
- removed joint Torso_Head
- added joint 0_1: type revolute, parent 0, child 1, origin xyz=2.699314353951913 0 0 rpy=0 0 0, axis 0 1 0, limit lower=-3.14159 upper=3.14159 effort=0.0 velocity=0.0
- added joint 1_2: type revolute, parent 1, child 2, origin xyz=1.8775634867757782 0 0 rpy=0 0 0, axis 0 1 0, limit lower=-3.14159 upper=3.14159 effort=0.0 velocity=0.0
- added joint 2_3: type revolute, parent 2, child 3, origin xyz=2.0000962611517035 0 0 rpy=0 0 0, axis 0 1 0, limit lower=-3.14159 upper=3.14159 effort=0.0 velocity=0.0
- added joint Head_0: type revolute, parent Head, child 0, origin xyz=0.17049013128728985 0 1.5 rpy=0 0 0, axis 0 1 0, limit lower=-3.14159 upper=3.14159 effort=0.0 velocity=0.0
